Commit message: Internal Communication rewritten plus start of robotarm

File: DEV/ROS/catkin_ws/src/ibo1_irc_api/description/external_camera.xacro (robot description, xacro)
@@ -37,4 +37,10 @@
     </joint>
     <link name="ec_camera_link"/>
+    <joint name="ec_color_module" type="fixed">
+        <origin xyz="0 0 0" rpy="${-pi/2} 0 ${-pi/2}" />
+        <parent link="ec_camera_link" />
+        <child  link="ec_color_frame" />
+    </joint>
+    <link name="ec_color_frame" />
     <joint name="ec_depth_module" type="fixed">
         <origin xyz="0 0.0125 0" rpy="${-pi/2} 0 ${-pi/2}" />
@@ -43,10 +49,4 @@
     </joint>
     <link name="ec_depth_frame"/>
-    <joint name="ec_color_module" type="fixed">
-        <origin xyz="0 0 0" rpy="${-pi/2} 0 ${-pi/2}" />
-        <parent link="ec_camera_link" />
-        <child  link="ec_color_frame" />
-    </joint>
-    <link name="ec_color_frame" />
     <!-- Cameras-->
     <xacro:property name="deg_to_rad" value="0.01745329251994329577" />

Commit message: Friday update

File: DEV/ROS/catkin_ws/src/ibo1_irc_api/description/external_camera.xacro (robot description, xacro)
@@ -9,5 +9,5 @@
         <child link="ec_base_link" />
         <parent link="world" />
-        <origin xyz="-0.25 0.5 1" rpy="0 0 0" />
+        <origin xyz="0 0.35 1" rpy="0 0 0" />
     </joint>
     <link name="ec_base_link">
